File: 555_doom_kicad/555_doom_kicad.kicad_sch (KiCad schematic)
At the start: 89 parts, among them J1 Power, J2 Speaker Out, Q1 2N3904, Q2 2N3904, SW1 SW_Push, U1 NE555P, U2 74LS161, U3 74154, U4 74HC14, U5 CD4066BE, U6 CD4066BE, U7 NE555P, U8 LM386

Commit message: Add KiCad files.
Parts:
- RV8: value 10K Volume -> 100K Volume
Changed lines of the file:
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@@
 			)
 		)
-		(property "Value" "10K Volume"
+		(property "Value" "100K Volume"
 			(at 71.12 200.6599 0)
 			(show_name no)
